Commit message: 14/1

File: description/robot_core.xacro (robot description, xacro)
@@ -37,9 +37,9 @@
         <parent link="base_link"/>
         <child link="chassis"/>
-        <origin xyz="${-wheel_offset_x} 0 0"/>
+        <origin xyz="-${wheel_offset_x} 0 0"/>
     </joint>
     <link name="chassis">
         <visual>
-            <origin xyz="${chassis_radius} 0 ${chassis_height/2 - 0.005}"/>
+            <origin xyz="${chassis_radius} 0 ${chassis_height/2}"/>
             <geometry>
                 <cylinder radius="${chassis_radius}" length="${chassis_height}"/>
@@ -48,5 +48,5 @@
         </visual>
         <collision>
-            <origin xyz="${chassis_radius} 0 ${chassis_height/2 - 0.005}"/>
+            <origin xyz="${chassis_radius} 0 ${chassis_height/2}"/>
             <geometry>
                 <cylinder radius="${chassis_radius}" length="${chassis_height}"/>
@@ -54,6 +54,6 @@
         </collision>
         <xacro:inertial_cylinder mass="${chassis_mass}" length="${chassis_height}" radius="${chassis_radius}">
-            <origin xyz="${chassis_radius} 0 ${chassis_height/2 - 0.005}" rpy="0 0 0"/>
-        </xacro:inertial_box>
+            <origin xyz="${chassis_radius} 0 ${chassis_height/2}" rpy="0 0 0"/>
+        </xacro:inertial_cylinder>
     </link>
     <!-- LEFT WHEEL LINK -->
@@ -81,8 +81,8 @@
     </link>
     <!-- RIGHT WHEEL LINK -->
-    <joint name="right_wheel_joint" type="continuous">
+   <joint name="right_wheel_joint" type="continuous">
         <parent link="base_link"/>
         <child link="right_wheel"/>
-        <origin xyz="0 ${-wheel_offset_y} ${wheel_offset_z}" rpy="${pi/2} 0 0" />
+        <origin xyz="0 -${wheel_offset_y} ${wheel_offset_z}" rpy="${pi/2} 0 0" />
         <axis xyz="0 0 -1"/>
     </joint>
@@ -106,5 +106,5 @@
     <joint name="caster_before_wheel_joint" type="fixed">
         <parent link="chassis"/>
-        <child link="caster_wheel"/>
+        <child link="caster_before_wheel"/>
         <origin xyz="${caster_wheel_offset_x} 0 ${caster_wheel_offset_z}"/>
     </joint>
@@ -127,6 +127,6 @@
     <joint name="caster_after_wheel_joint" type="fixed">
         <parent link="chassis"/>
-        <child link="caster_wheel"/>
-        <origin xyz="$0.0375 0 ${caster_wheel_offset_z}"/>
+        <child link="caster_after_wheel"/>
+        <origin xyz="0.0375 0 ${caster_wheel_offset_z}"/>
     </joint>
     <link name="caster_after_wheel">

Commit message: update 14/1

File: description/robot_core.xacro (robot description, xacro)
@@ -14,5 +14,5 @@
     <xacro:property name="caster_wheel_mass" value="0.01"/>
     <xacro:property name="caster_wheel_offset_x" value="0.3125"/> <!-- x = 137.5 + 175mm-->
-    <xacro:property name="caster_wheel_offset_z" value="-0.015"/> <!-- z = 15mm-->
+    <xacro:property name="caster_wheel_offset_z" value="-0.01"/> <!-- z = 10mm-->
     <material name="white">
         <color rgba="1 1 1 1" />
@@ -32,4 +32,7 @@
     <!-- BASE LINK -->
     <link name="base_link">
+      <visual>
+        <origin xyz="0 0 0.015" rpy="0 0 0" />
+      </visual>
     </link>
     <!-- CHASSIS LINK -->
@@ -41,5 +44,5 @@
     <link name="chassis">
         <visual>
-            <origin xyz="${chassis_radius} 0 ${chassis_height/2}"/>
+            <origin xyz="${chassis_radius} 0 ${chassis_height/2 - 0.005}"/>
             <geometry>
                 <cylinder radius="${chassis_radius}" length="${chassis_height}"/>
@@ -48,5 +51,5 @@
         </visual>
         <collision>
-            <origin xyz="${chassis_radius} 0 ${chassis_height/2}"/>
+            <origin xyz="${chassis_radius} 0 ${chassis_height/2 - 0.005}"/>
             <geometry>
                 <cylinder radius="${chassis_radius}" length="${chassis_height}"/>
@@ -54,5 +57,5 @@
         </collision>
         <xacro:inertial_cylinder mass="${chassis_mass}" length="${chassis_height}" radius="${chassis_radius}">
-            <origin xyz="${chassis_radius} 0 ${chassis_height/2}" rpy="0 0 0"/>
+            <origin xyz="${chassis_radius} 0 ${chassis_height/2 - 0.005}" rpy="0 0 0"/>
         </xacro:inertial_cylinder>
     </link>

Commit message: Update robot_core.xacro

File: description/robot_core.xacro (robot description, xacro)
@@ -3,5 +3,5 @@
     <xacro:include filename="inertial_macros.xacro"/>
     <xacro:property name="chassis_radius" value="0.175"/> <!-- R = 175mm-->
-    <xacro:property name="chassis_height" value="0.12"/> <!-- h = 120mm-->
+    <xacro:property name="chassis_height" value="0.125"/> <!-- h = 125mm-->
     <xacro:property name="chassis_mass" value="1.0"/>
     <xacro:property name="wheel_radius" value="0.0325"/> <!-- R = 32.5mm-->
@@ -9,9 +9,9 @@
     <xacro:property name="wheel_mass" value="0.05"/>
     <xacro:property name="wheel_offset_x" value="0.175"/> <!-- x = 175mm-->
-    <xacro:property name="wheel_offset_y" value="0.133"/> <!-- y = 120mm + 12.5mm + 0.5mm-->
+    <xacro:property name="wheel_offset_y" value="0.1425"/> <!-- y = 142.5mm-->
     <xacro:property name="wheel_offset_z" value="0.0125"/> <!-- z = 12.5mm-->
     <xacro:property name="caster_wheel_radius" value="0.01"/>  <!-- R = 10mm-->
     <xacro:property name="caster_wheel_mass" value="0.01"/>
-    <xacro:property name="caster_wheel_offset_x" value="0.3125"/> <!-- x = 137.5 + 175mm-->
+    <xacro:property name="caster_wheel_offset_x" value="0.32"/> <!-- x = 145 + 175mm-->
     <xacro:property name="caster_wheel_offset_z" value="-0.01"/> <!-- z = 10mm-->
     <material name="white">
@@ -131,5 +131,5 @@
         <parent link="chassis"/>
         <child link="caster_after_wheel"/>
-        <origin xyz="0.0375 0 ${caster_wheel_offset_z}"/>
+        <origin xyz="0.03 0 ${caster_wheel_offset_z}"/>
     </joint>
     <link name="caster_after_wheel">

Commit message: Update robot_core.xacro

File: description/robot_core.xacro (robot description, xacro)
@@ -3,5 +3,5 @@
     <xacro:include filename="inertial_macros.xacro"/>
     <xacro:property name="chassis_radius" value="0.175"/> <!-- R = 175mm-->
-    <xacro:property name="chassis_height" value="0.125"/> <!-- h = 125mm-->
+    <xacro:property name="chassis_height" value="0.005"/> <!-- h = 5mm-->
     <xacro:property name="chassis_mass" value="1.0"/>
     <xacro:property name="wheel_radius" value="0.0325"/> <!-- R = 32.5mm-->
@@ -44,12 +44,51 @@
     <link name="chassis">
         <visual>
-            <origin xyz="${chassis_radius} 0 ${chassis_height/2 - 0.005}"/>
+            <origin xyz="${chassis_radius} 0 -${chassis_height/2}"/>
             <geometry>
                 <cylinder radius="${chassis_radius}" length="${chassis_height}"/>
             </geometry>
-            <material name="white"/>
+            <material name="orange"/>
+        </visual>
+        <visual>
+            <origin xyz="${chassis_radius} 0 0.13"/>
+            <geometry>
+                <cylinder radius="${chassis_radius}" length="${chassis_height}"/>
+            </geometry>
+            <material name="orange"/>
+        </visual>
+        <!-- Tru 1 -->
+        <visual>
+            <origin xyz="0.035 0.05799 0.0625"/>
+            <geometry>
+                <cylinder radius="0.008" length="0.125"/>
+            </geometry>
+            <material name="black"/>
+        </visual>
+        <!-- Tru 2 -->
+        <visual>
+            <origin xyz="0.035 -0.05799 0.0625"/>
+            <geometry>
+                <cylinder radius="0.008" length="0.125"/>
+            </geometry>
+            <material name="black"/>
+        </visual>
+        <!-- Tru 3 -->
+        <visual>
+            <origin xyz="0.315 0.05799 0.0625"/>
+            <geometry>
+                <cylinder radius="0.008" length="0.125"/>
+            </geometry>
+            <material name="black"/>
+        </visual>
+        <!-- Tru 4 -->
+        <visual>
+            <origin xyz="0.315 -0.05799 0.0625"/>
+            <geometry>
+                <cylinder radius="0.008" length="0.125"/>
+            </geometry>
+            <material name="black"/>
         </visual>
         <collision>
-            <origin xyz="${chassis_radius} 0 ${chassis_height/2 - 0.005}"/>
+            <origin xyz="${chassis_radius} 0 -${chassis_height/2}"/>
             <geometry>
                 <cylinder radius="${chassis_radius}" length="${chassis_height}"/>
@@ -57,5 +96,5 @@
         </collision>
         <xacro:inertial_cylinder mass="${chassis_mass}" length="${chassis_height}" radius="${chassis_radius}">
-            <origin xyz="${chassis_radius} 0 ${chassis_height/2 - 0.005}" rpy="0 0 0"/>
+            <origin xyz="${chassis_radius} 0 -${chassis_height/2}" rpy="0 0 0"/>
         </xacro:inertial_cylinder>
     </link>

Commit message: Update robot_core.xacro

File: description/robot_core.xacro (robot description, xacro)
@@ -95,6 +95,13 @@
             </geometry>
         </collision>
+        <collision>
+            <origin xyz="${chassis_radius} 0 0.13"/>
+            <geometry>
+                <cylinder radius="${chassis_radius}" length="${chassis_height}"/>
+            </geometry>
+        </collision>
         <xacro:inertial_cylinder mass="${chassis_mass}" length="${chassis_height}" radius="${chassis_radius}">
             <origin xyz="${chassis_radius} 0 -${chassis_height/2}" rpy="0 0 0"/>
+            <origin xyz="${chassis_radius} 0 0.13" rpy="0 0 0"/>
         </xacro:inertial_cylinder>
     </link>

Commit message: Update robot_core.xacro

File: description/robot_core.xacro (robot description, xacro)
@@ -63,5 +63,5 @@
                 <cylinder radius="0.008" length="0.125"/>
             </geometry>
-            <material name="black"/>
+            <material name="orange"/>
         </visual>
         <!-- Tru 2 -->
@@ -71,5 +71,5 @@
                 <cylinder radius="0.008" length="0.125"/>
             </geometry>
-            <material name="black"/>
+            <material name="orange"/>
         </visual>
         <!-- Tru 3 -->
@@ -79,5 +79,5 @@
                 <cylinder radius="0.008" length="0.125"/>
             </geometry>
-            <material name="black"/>
+            <material name="orange"/>
         </visual>
         <!-- Tru 4 -->
@@ -87,5 +87,5 @@
                 <cylinder radius="0.008" length="0.125"/>
             </geometry>
-            <material name="black"/>
+            <material name="orange"/>
         </visual>
         <collision>
