Commit message: Update lidar.xacro

File: description/lidar.xacro (robot description, xacro)
@@ -4,12 +4,19 @@
         <parent link="chassis"/>
         <child link="laser_frame"/>
-        <origin xyz="0.2617 0 0.134" rpy="0 0 0"/>
+        <origin xyz="0.2666 0 0.161" rpy="0 0 0"/> <--! h = 125mm + 5mm + 31mm + 12mm -->
     </joint>
     <link name="laser_frame">
         <visual>
             <geometry>
-                <cylinder radius="0.035" length="0.028"/>
+                <cylinder radius="0.035" length="0.024"/>
             </geometry>
             <material name="red"/>
+        </visual>
+         <visual>
+            <origin xyz="0 0 -0.0275"/>
+            <geometry>
+                <cylinder radius="0.004" length="0.031"/>
+            </geometry>
+            <material name="black"/>
         </visual>
         <collision>

Commit message: Update lidar.xacro

File: description/lidar.xacro (robot description, xacro)
@@ -22,8 +22,8 @@
         <collision>
             <geometry>
-                <cylinder radius="0.035" length="0.028"/>
+                <cylinder radius="0.035" length="0.024"/>
             </geometry>
         </collision>
-        <xacro:inertial_cylinder mass="0.1" length="0.028" radius="0.035">
+        <xacro:inertial_cylinder mass="0.1" length="0.024" radius="0.035">
             <origin xyz="0 0 0" rpy="0 0 0"/>
         </xacro:inertial_cylinder>

Commit message: 20/1

File: description/lidar.xacro (robot description, xacro)
@@ -4,5 +4,5 @@
         <parent link="chassis"/>
         <child link="laser_frame"/>
-        <origin xyz="0.2666 0 0.161" rpy="0 0 0"/> <--! h = 125mm + 5mm + 31mm + 12mm -->
+        <origin xyz="0.2666 0 0.173" rpy="0 0 0"/> <!-- h = 125mm + 5mm + 31mm + 12mm -->
     </joint>
     <link name="laser_frame">
@@ -18,5 +18,5 @@
                 <cylinder radius="0.004" length="0.031"/>
             </geometry>
-            <material name="black"/>
+            <material name="white"/>
         </visual>
         <collision>

File: description/robot_core.xacro (robot description, xacro)
@@ -51,5 +51,5 @@
         </visual>
         <visual>
-            <origin xyz="${chassis_radius} 0 0.13"/>
+            <origin xyz="${chassis_radius} 0 0.1275"/>
             <geometry>
                 <cylinder radius="${chassis_radius}" length="${chassis_height}"/>
@@ -96,5 +96,5 @@
         </collision>
         <collision>
-            <origin xyz="${chassis_radius} 0 0.13"/>
+            <origin xyz="${chassis_radius} 0 0.1275"/>
             <geometry>
                 <cylinder radius="${chassis_radius}" length="${chassis_height}"/>
@@ -103,5 +103,7 @@
         <xacro:inertial_cylinder mass="${chassis_mass}" length="${chassis_height}" radius="${chassis_radius}">
             <origin xyz="${chassis_radius} 0 -${chassis_height/2}" rpy="0 0 0"/>
-            <origin xyz="${chassis_radius} 0 0.13" rpy="0 0 0"/>
+        </xacro:inertial_cylinder>
+         <xacro:inertial_cylinder mass="${chassis_mass}" length="${chassis_height}" radius="${chassis_radius}">
+            <origin xyz="${chassis_radius} 0 0.1275" rpy="0 0 0"/>
         </xacro:inertial_cylinder>
     </link>

Commit message: Update lidar.xacro

File: description/lidar.xacro (robot description, xacro)
@@ -11,5 +11,5 @@
                 <cylinder radius="0.035" length="0.024"/>
             </geometry>
-            <material name="red"/>
+            <material name="black"/>
         </visual>
          <visual>
@@ -18,5 +18,5 @@
                 <cylinder radius="0.004" length="0.031"/>
             </geometry>
-            <material name="white"/>
+            <material name="black"/>
         </visual>
         <collision>
